Commit message: Update turtlebot3_waffle.urdf

File: nav2_bringup/urdf/turtlebot3_waffle.urdf (robot description, URDF)
Before this commit: robot turtlebot3_waffle, 13 links, 12 joints
Links:
- removed link base_scan
- removed link camera_depth_frame
- removed link camera_depth_optical_frame
- removed link camera_link
- removed link camera_rgb_frame
- removed link camera_rgb_optical_frame
- removed link caster_back_left_link
- removed link caster_back_right_link
- removed link imu_link
- removed link wheel_left_link
- removed link wheel_right_link
- added link l_back_wheel; collision cylinder length=0.025 radius=0.03; visual cylinder length=0.025 radius=0.03
- added link l_front_wheel; collision cylinder length=0.025 radius=0.03; visual cylinder length=0.025 radius=0.03
- added link laser; collision cylinder length=0.06 radius=0.035; visual cylinder length=0.06 radius=0.035
- added link r_back_wheel; collision cylinder length=0.025 radius=0.03; visual cylinder length=0.025 radius=0.03
- added link r_front_wheel; collision cylinder length=0.025 radius=0.03; visual cylinder length=0.025 radius=0.03
- link base_link: mass 1.3729096e+00 -> None; geometry collision box size=0.3 0.26 0.1; visual box size=0.245 0.1 0.225
Joints:
- removed joint base_joint
- removed joint camera_depth_joint
- removed joint camera_depth_optical_joint
- removed joint camera_joint
- removed joint camera_rgb_joint
- removed joint camera_rgb_optical_joint
- removed joint caster_back_left_joint
- removed joint caster_back_right_joint
- removed joint imu_joint
- removed joint scan_joint
- removed joint wheel_left_joint
- removed joint wheel_right_joint
- added joint base_footprint_fixed: type fixed, parent base_footprint, child base_link, origin xyz=0 0 0 rpy=0 0 0
- added joint base_link_fixed: type fixed, parent base_link, child laser, origin xyz=0 0 0 rpy=0 0 0
- added joint l_back_wheel_joint: type continuous, parent base_link, child l_back_wheel, origin xyz=-0.0925 -0.0625 0.03 rpy=1.570796 0 0, axis 0 1 0
- added joint l_front_wheel_joint: type continuous, parent base_link, child l_front_wheel, origin xyz=-0.0925 0.0625 0.03 rpy=1.570796 0 0, axis 0 1 0
- added joint laser: type continuous, parent base_link, child laser, origin xyz=0 0 0 rpy=0 0 0, axis 0 1 0
- added joint r_back_wheel_joint: type continuous, parent base_link, child r_back_wheel, origin xyz=0.0925 -0.0625 0.03 rpy=1.570796 0 0, axis 0 1 0
- added joint r_front_wheel_joint: type continuous, parent base_link, child r_front_wheel, origin xyz=0.0925 0.0625 0.03 rpy=1.570796 0 0, axis 0 1 0

Commit message: Update turtlebot3_waffle.urdf

File: nav2_bringup/urdf/turtlebot3_waffle.urdf (robot description, URDF)
Before this commit: robot turtlebot3_waffle, 7 links, 7 joints
Links:
- link base_link: geometry collision box size=0.10 0.195 0.225; visual box size=0.10 0.195 0.225

Commit message: Update turtlebot3_waffle.urdf

File: nav2_bringup/urdf/turtlebot3_waffle.urdf (robot description, URDF)
Before this commit: robot turtlebot3_waffle, 7 links, 7 joints
Links:
- link l_back_wheel: geometry collision cylinder length=0.025 radius=0.035; visual cylinder length=0.025 radius=0.035
- link l_front_wheel: geometry collision cylinder length=0.025 radius=0.035; visual cylinder length=0.025 radius=0.035
- link r_back_wheel: geometry collision cylinder length=0.025 radius=0.035; visual cylinder length=0.025 radius=0.035
- link r_front_wheel: geometry collision cylinder length=0.025 radius=0.035; visual cylinder length=0.025 radius=0.035
Joints:
- removed joint base_link_fixed
- joint base_footprint_fixed: origin xyz=0 0 0 rpy=0 0 0 -> xyz=0 0 0.015 rpy=0 0 0
- joint l_back_wheel_joint: origin xyz=-0.0925 -0.0625 0.03 rpy=1.570796 0 0 -> xyz=0.0925 0.0625 0.03 rpy=1.570796 0 0
- joint laser: origin xyz=0 0 0 rpy=0 0 0 -> xyz=0 0 0.3 rpy=0 0 0
- joint r_front_wheel_joint: origin xyz=0.0925 0.0625 0.03 rpy=1.570796 0 0 -> xyz=-0.0925 -0.0625 0.03 rpy=1.570796 0 0

Commit message: Update turtlebot3_waffle.urdf

File: nav2_bringup/urdf/turtlebot3_waffle.urdf (robot description, URDF)
Before this commit: robot turtlebot3_waffle, 7 links, 6 joints
Links:
- added link box_link; visual box size=0.10 0.195 0.255
- link base_link: geometry collision box ; visual box 
Joints:
- added joint box_joint: type fixed, parent base_link, child box_link, origin xyz=-0.1 0 0
- joint l_back_wheel_joint: origin xyz=0.0925 0.0625 0.03 rpy=1.570796 0 0 -> xyz=-0.0575 -0.0675 0.035 rpy=1.570796 0 0
- joint l_front_wheel_joint: origin xyz=-0.0925 0.0625 0.03 rpy=1.570796 0 0 -> xyz=0.0575 -0.0675 0.035 rpy=1.570796 0 0
- joint r_back_wheel_joint: origin xyz=0.0925 -0.0625 0.03 rpy=1.570796 0 0 -> xyz=-0.0575 0.0675 0.035 rpy=1.570796 0 0
- joint r_front_wheel_joint: origin xyz=-0.0925 -0.0625 0.03 rpy=1.570796 0 0 -> xyz=0.0575 0.0675 0.035 rpy=1.570796 0 0
